File: weatherstation.sch (EAGLE design)
At the start: 62 parts, among them CON1 USBC, CON2 DC-005, CON3 LCD-TFT, CON4 ST-LINK, CON5 TEST, CON6 BME680, T1 2N7002, T2 2N7002, T3 2N7002, T4 2N7002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

Commit message: Changing wrong rev
Other:
- note added: "1.0"
- note removed: "2.4"
Changed lines of the file:
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@@
 <text x="152.4" y="121.92" size="2.54" layer="94">Buttons</text>
 <text x="72.136" y="39.116" size="1.6764" layer="94">ammeter con</text>
-<text x="314.706" y="5.08" size="2.54" layer="94">2.4</text>
+<text x="314.706" y="5.08" size="2.54" layer="94">1.0</text>
 <text x="149.86" y="185.42" size="2.54" layer="94">Connectors</text>
 <text x="5.08" y="116.84" size="2.54" layer="94">Power Indicator</text>
@@
 <wire x1="146.05" y1="127.254" x2="322.58" y2="127.254" width="0.1524" layer="94"/>
 <wire x1="146.05" y1="190.5" x2="322.58" y2="190.5" width="0.1524" layer="94"/>
-<text x="119.126" y="5.08" size="2.54" layer="94">2.4</text>
+<text x="119.126" y="5.08" size="2.54" layer="94">1.0</text>
 <text x="283.464" y="10.16" size="2.54" layer="94">29.09.2024</text>
 <text x="87.63" y="10.16" size="2.54" layer="94">29.09.2024</text>
